File: gingham.kicad_pcb (KiCad board)
At the start: 2 copper layers, 285.8 x 123.8 mm, 167 parts, among them J1 Molex-0548190519, J2 ISP, SW1 SW_Push, SW10 SW_Push, SW11 SW_Push, SW12 SW_Push, SW13 SW_Push, SW14 SW_Push, SW15 SW_Push, SW16 SW_Push, SW17 SW_Push, SW18 SW_Push, SW19 SW_Push, SW2 SW_Push, SW20 SW_Push, SW21 SW_Push, SW22 SW_Push, SW23 SW_Push, SW24 SW_Push, SW25 SW_Push, SW26 SW_Push, SW27 SW_Push, SW28 SW_Push, SW29 SW_Push, SW3 SW_Push, SW30 SW_Push, SW31 SW_Push, SW32 SW_Push, SW33 SW_Push, SW34 SW_Push, SW35 SW_Push, SW36 SW_Push, SW37 SW_Push, SW38 SW_Push, SW39 SW_Push, SW4 SW_Push, SW40 SW_Push, SW41 SW_Push, SW42 SW_Push, SW43 SW_Push, SW44 SW_Push, SW45 SW_Push, SW46 SW_Push, SW47 SW_Push, SW48 SW_Push, SW49 SW_Push, SW5 SW_Push, SW50 SW_Push, SW51 SW_Push, SW52 SW_Push, SW53 SW_Push, SW54 SW_Push, SW55 SW_Push, SW56 SW_Push, SW57 SW_Push, SW58 SW_Push, SW59 SW_Push, SW6 SW_Push, SW60 SW_Push, SW61 SW_Push, SW62 SW_Push, SW63 SW_Push, SW64 SW_Push, SW65 SW_Push, SW66 SW_Push, SW67 SW_Push, SW68 RESET, SW69 BOOT, SW7 SW_Push, SW70 SW_Push, SW71 SW_Push, SW8 SW_Push, SW9 SW_Push, U1 ATMEGA328-PU, Y1 16MHz

Commit message: Add files via upload
Routing:
- net Net-(D161-Pad2): track 0.00 -> 46.9 mm
Changed lines of the file:
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@@
-(kicad_pcb (version 20190905) (host pcbnew "5.99.0-unknown-3cd1208~86~ubuntu18.04.1")
+(kicad_pcb (version 20190905) (host pcbnew "5.99.0-unknown-281d77f~86~ubuntu18.04.1")
   (general
     (thickness 1.6)
     (drawings 13)
-    (tracks 1513)
+    (tracks 1521)
     (modules 167)
     (nets 97)
@@
       (drillshape 0)
       (scaleselection 1)
-      (outputdirectory "gerbers/front/")
+      (outputdirectory "gerbers/")
     )
   )
@@
   (gr_line (start 330.9875 166.68125) (end 330.9875 47.61875) (layer "Edge.Cuts") (width 0.15))
   (gr_line (start 47.61875 169.0625) (end 328.60625 169.0625) (layer "Edge.Cuts") (width 0.15))
+  (segment (start 55 79.8) (end 58.149999 82.949999) (width 0.3) (layer "B.Cu") (net 96))
+  (segment (start 58.149999 82.949999) (end 58.149999 97.412501) (width 0.3) (layer "B.Cu") (net 96))
+  (segment (start 58.149999 97.412501) (end 55.715 99.8475) (width 0.3) (layer "B.Cu") (net 96))
+  (segment (start 55 77) (end 55 79.8) (width 0.3) (layer "B.Cu") (net 96))
+  (segment (start 56.4 75.6) (end 55 77) (width 0.3) (layer "B.Cu") (net 96))
+  (segment (start 59.95137 75.6) (end 56.4 75.6) (width 0.3) (layer "B.Cu") (net 96))
+  (segment (start 70.6 63.82) (end 70.6 64.95137) (width 0.3) (layer "B.Cu") (net 96))
+  (segment (start 70.6 64.95137) (end 59.95137 75.6) (width 0.3) (layer "B.Cu") (net 96))
   (via (at 311 94) (size 1) (drill 0.6) (layers "F.Cu" "B.Cu") (net 1))
   (via (at 311 112) (size 1) (drill 0.6) (layers "F.Cu" "B.Cu") (net 1))

Commit message: Add files via upload
Routing:
- net +5V: track 80.0 -> 83.0 mm
- net GND: vias 68 -> 91
- net (no net): vias 0 -> 3
Changed lines of the file:
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@@
     (thickness 1.6)
     (drawings 13)
-    (tracks 1521)
+    (tracks 1554)
     (modules 167)
     (nets 97)
@@
   (gr_line (start 330.9875 166.68125) (end 330.9875 47.61875) (layer "Edge.Cuts") (width 0.15))
   (gr_line (start 47.61875 169.0625) (end 328.60625 169.0625) (layer "Edge.Cuts") (width 0.15))
+  (via (at 298.2 47.2) (size 1) (drill 0.6) (layers "F.Cu" "B.Cu") (net 0))
+  (via (at 279.4 46.8) (size 1) (drill 0.6) (layers "F.Cu" "B.Cu") (net 0))
+  (via (at 286.6 54.6) (size 1) (drill 0.6) (layers "F.Cu" "B.Cu") (net 0))
+  (segment (start 289.5625 50.6875) (end 290.360405 50.6875) (width 0.3) (layer "B.Cu") (net 65))
+  (segment (start 290.360405 50.6875) (end 290.777916 50.269989) (width 0.3) (layer "B.Cu") (net 65))
+  (segment (start 290.777916 50.269989) (end 297.269989 50.269989) (width 0.3) (layer "B.Cu") (net 65))
+  (segment (start 297.269989 50.269989) (end 298.900001 51.900001) (width 0.3) (layer "B.Cu") (net 65))
+  (segment (start 298.900001 51.900001) (end 299.6 52.6) (width 0.3) (layer "B.Cu") (net 65))
+  (segment (start 305 54.5) (end 305 55.6) (width 0.3) (layer "B.Cu") (net 65))
+  (segment (start 303.1 52.6) (end 305 54.5) (width 0.3) (layer "B.Cu") (net 65))
+  (segment (start 299.6 52.6) (end 303.1 52.6) (width 0.3) (layer "B.Cu") (net 65))
+  (segment (start 296.8 52.6) (end 295.319999 51.119999) (width 0.8) (layer "B.Cu") (net 58))
+  (segment (start 295.319999 51.119999) (end 291.130001 51.119999) (width 0.8) (layer "B.Cu") (net 58))
+  (segment (start 291.130001 51.119999) (end 290.3625 51.8875) (width 0.8) (layer "B.Cu") (net 58))
+  (segment (start 280.87 57.55625) (end 280.87 60.09) (width 0.8) (layer "F.Cu") (net 57))
+  (segment (start 280.87 60.09) (end 280.98 60.2) (width 0.8) (layer "F.Cu") (net 57))
+  (segment (start 296.8 57.6) (end 295.399999 56.199999) (width 0.8) (layer "F.Cu") (net 57))
+  (segment (start 295.399999 56.199999) (end 282.226251 56.199999) (width 0.8) (layer "F.Cu") (net 57))
+  (segment (start 282.226251 56.199999) (end 281.669999 56.756251) (width 0.8) (layer "F.Cu") (net 57))
+  (segment (start 281.669999 56.756251) (end 280.87 57.55625) (width 0.8) (layer "F.Cu") (net 57))
+  (segment (start 299.6 57.68) (end 302.28 57.68) (width 0.8) (layer "F.Cu") (net 57))
+  (segment (start 302.28 57.68) (end 303 58.4) (width 0.8) (layer "F.Cu") (net 57))
+  (segment (start 296.8 57.6) (end 299.52 57.6) (width 0.8) (layer "F.Cu") (net 57))
+  (segment (start 299.52 57.6) (end 299.6 57.68) (width 0.8) (layer "F.Cu") (net 57))
   (segment (start 55 79.8) (end 58.149999 82.949999) (width 0.3) (layer "B.Cu") (net 96))
   (segment (start 58.149999 82.949999) (end 58.149999 97.412501) (width 0.3) (layer "B.Cu") (net 96))
@@
   (segment (start 230.054374 163) (end 171.6 163) (width 0.3) (layer "B.Cu") (net 50))
   (segment (start 171.6 163) (end 163.6375 155.0375) (width 0.3) (layer "B.Cu") (net 50))
-  (segment (start 296.8 57.6) (end 299.52 57.6) (width 0.3) (layer "F.Cu") (net 57))
-  (segment (start 299.6 57.68) (end 300.32 58.4) (width 0.3) (layer "F.Cu") (net 57))
-  (segment (start 300.32 58.4) (end 303 58.4) (width 0.3) (layer "F.Cu") (net 57))
   (segment (start 313.94 49) (end 313.94 64.08) (width 0.3) (layer "F.Cu") (net 61))
   (segment (start 313.94 64.08) (end 315.63 65.77) (width 0.3) (layer "F.Cu") (net 61))
@@
   (segment (start 291.2 57.6) (end 288.6 60.2) (width 0.3) (layer "B.Cu") (net 46))
   (segment (start 294 57.6) (end 291.2 57.6) (width 0.3) (layer "B.Cu") (net 46))
-  (segment (start 290.880001 51.369999) (end 290.3625 51.8875) (width 0.3) (layer "B.Cu") (net 58))
-  (segment (start 295.569999 51.369999) (end 290.880001 51.369999) (width 0.3) (layer "B.Cu") (net 58))
-  (segment (start 296.8 52.6) (end 295.569999 51.369999) (width 0.3) (layer "B.Cu") (net 58))
-  (segment (start 297.6875 50.6875) (end 289.5625 50.6875) (width 0.3) (layer "B.Cu") (net 65))
-  (segment (start 299.6 52.6) (end 297.6875 50.6875) (width 0.3) (layer "B.Cu") (net 65))
   (segment (start 288.376717 49.16249) (end 286.95751 49.16249) (width 0.3) (layer "B.Cu") (net 65))
   (segment (start 283.6 52.52) (end 286.95751 49.16249) (width 0.3) (layer "B.Cu") (net 65))
   (segment (start 289.5625 50.348273) (end 288.376717 49.16249) (width 0.3) (layer "B.Cu") (net 65))
-  (segment (start 305 54.5) (end 305 55.6) (width 0.3) (layer "B.Cu") (net 65))
-  (segment (start 303.1 52.6) (end 305 54.5) (width 0.3) (layer "B.Cu") (net 65))
-  (segment (start 299.6 52.6) (end 303.1 52.6) (width 0.3) (layer "B.Cu") (net 65))
   (segment (start 297.08 55.6) (end 294 52.52) (width 0.3) (layer "B.Cu") (net 66))
   (segment (start 302.2 55.6) (end 297.08 55.6) (width 0.3) (layer "B.Cu") (net 66))
@@
   (segment (start 280.98 67.82) (end 280.98 70.29137) (width 0.3) (layer "B.Cu") (net 1))
   (segment (start 275.9 67.82) (end 275.9 70.37137) (width 0.3) (layer "B.Cu") (net 57))
-  (segment (start 295.649999 56.449999) (end 296.8 57.6) (width 0.3) (layer "F.Cu") (net 57))
-  (segment (start 281.976251 56.449999) (end 295.649999 56.449999) (width 0.3) (layer "F.Cu") (net 57))
-  (segment (start 280.87 57.55625) (end 281.976251 56.449999) (width 0.3) (layer "F.Cu") (net 57))
   (segment (start 323.196251 101.883751) (end 319.2 97.8875) (width 0.3) (layer "B.Cu") (net 56))
   (segment (start 180 69.454374) (end 180 55.22) (width 0.3) (layer "B.Cu") (net 78))
@@
   (segment (start 259.4 98.8) (end 259.4 96.6) (width 0.3) (layer "B.Cu") (net 78))
   (segment (start 248.4 81) (end 249.8 79.6) (width 0.3) (layer "B.Cu") (net 78))
+  (via (at 53.8 127.2) (size 1) (drill 0.6) (layers "F.Cu" "B.Cu") (net 1))
+  (via (at 53.6 93.6) (size 1) (drill 0.6) (layers "F.Cu" "B.Cu") (net 1))
+  (via (at 59.6 91.4) (size 1) (drill 0.6) (layers "F.Cu" "B.Cu") (net 1))
+  (via (at 59 74.2) (size 1) (drill 0.6) (layers "F.Cu" "B.Cu") (net 1))
+  (via (at 64.6 111) (size 1) (drill 0.6) (layers "F.Cu" "B.Cu") (net 1))
+  (via (at 263.4 107.8) (size 1) (drill 0.6) (layers "F.Cu" "B.Cu") (net 1))
+  (via (at 227.6 109.6) (size 1) (drill 0.6) (layers "F.Cu" "B.Cu") (net 1))
+  (via (at 258.8 142.8) (size 1) (drill 0.6) (layers "F.Cu" "B.Cu") (net 1))
+  (via (at 234.4 159.8) (size 1) (drill 0.6) (layers "F.Cu" "B.Cu") (net 1))
+  (via (at 129.6 98.4) (size 1) (drill 0.6) (layers "F.Cu" "B.Cu") (net 1))
+  (via (at 107.2 150.8) (size 1) (drill 0.6) (layers "F.Cu" "B.Cu") (net 1))
+  (via (at 109.2 130) (size 1) (drill 0.6) (layers "F.Cu" "B.Cu") (net 1))
+  (via (at 78.4 93.6) (size 1) (drill 0.6) (layers "F.Cu" "B.Cu") (net 1))
+  (via (at 55 111.6) (size 1) (drill 0.6) (layers "F.Cu" "B.Cu") (net 1))
+  (via (at 167 161.8) (size 1) (drill 0.6) (layers "F.Cu" "B.Cu") (net 1))
+  (via (at 173.8 126) (size 1) (drill 0.6) (layers "F.Cu" "B.Cu") (net 1))
+  (via (at 173.2 117.6) (size 1) (drill 0.6) (layers "F.Cu" "B.Cu") (net 1))
+  (via (at 156 116.8) (size 1) (drill 0.6) (layers "F.Cu" "B.Cu") (net 1))
+  (via (at 282.4 156.8) (size 1) (drill 0.6) (layers "F.Cu" "B.Cu") (net 1))
+  (via (at 259.8 155.6) (size 1) (drill 0.6) (layers "F.Cu" "B.Cu") (net 1))
+  (via (at 307.8 159.8) (size 1) (drill 0.6) (layers "F.Cu" "B.Cu") (net 1))
+  (via (at 301.4 99.4) (size 1) (drill 0.6) (layers "F.Cu" "B.Cu") (net 1))
+  (via (at 328.2 56.2) (size 1) (drill 0.6) (layers "F.Cu" "B.Cu") (net 1))
   (zone (net 1) (net_name "GND") (layer "F.Cu") (hatch edge 0.508)
     (connect_pads (clearance 0.508))

Commit message: Add files via upload
Parts:
- moved D48 13.2 mm to (60.2, 50.2)
- moved SW68 10.1 mm to (241.3, 50.5)
- moved SW69 9.75 mm to (231.3, 50.5)
- moved D2 7.87 mm to (73.2, 56.6)
- moved D3 3.75 mm to (94.2, 56.7)
- moved D4 3.68 mm to (91.6, 55.4)
- moved D47 3.00 mm to (62.8, 51.5)
- moved D46 2.86 mm to (65.4, 52.8)
- moved D53 2.62 mm to (138.4, 47.6)
- moved D54 2.62 mm to (141.0, 48.9)
- moved D67 2.62 mm to (203.4, 48.9)
- moved D60 2.60 mm to (55.0, 47.6)
- moved D61 2.60 mm to (57.6, 49.0)
- moved D66 2.60 mm to (200.8, 47.6)
- moved D17 2.10 mm to (89.0, 54.1)
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Routing:
- net Net-(D44-Pad2): track 188.2 -> 157.3 mm
- net Net-(D67-Pad2): track 211.1 -> 185.4 mm
- net /RESET: track 147.5 -> 122.2 mm
- net GND: track 18.4 -> 43.0 mm, vias 91 -> 72
- net /ROW3: track 290.5 -> 268.0 mm
- net Net-(D48-Pad2): track 100.5 -> 120.7 mm
- net Net-(D161-Pad2): track 46.9 -> 63.9 mm
- net Net-(D24-Pad2): track 102.8 -> 86.6 mm
- net Net-(D32-Pad2): track 81.8 -> 65.9 mm
- net /ROW0: track 282.0 -> 268.0 mm
- net Net-(D53-Pad2): track 118.5 -> 104.6 mm
- net Net-(D61-Pad2): track 138.3 -> 124.9 mm
- net /ROW5: track 202.3 -> 213.9 mm
- net Net-(D71-Pad2): track 122.3 -> 110.9 mm
- net /ROW2: track 219.4 -> 208.3 mm
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